File: 451.sch (KiCad schematic (older format))
At the start: 20 parts, among them U1 68010D, U2 68451, U3 74LS245, U4 74LS245, U5 74LS04, U6 74LS00, X1 8Mhz

Commit message: finish memory layout thing
Parts:
- removed unit 1 of U5
- removed unit 2 of U5
- removed unit 1 of U6
Connections:
- net AS is gone; now on net \AS: U1.6 (AS), U2.13 (AS)
- net MAS is gone; now on net \MAS: U2.2 (MAS)
- net \BG: now reaches U1.11 (BG)
- net \BGACK: now reaches U1.12 (BGACK)
- net \BR: now reaches U1.13 (BR)
- net \HALT: now reaches U1.17 (HALT)
- net \RST: now reaches U1.18 (RESET)
- net \RST: now also U2.14 (RESET)
- net \VMA: now reaches U1.19 (VMA)
- net E: now reaches U1.20 (E)
- net \VPA: now reaches U1.21 (VPA)
- net \BERR: now reaches U1.22 (BERR)
- net \BERR: now also U2.6 (FAULT)
- net \IPL2: now reaches U1.23 (IPL2)
- net \IPL1: now reaches U1.24 (IPL1)
- net \IPL0: now reaches U1.25 (IPL0)
- net \MMUSEL: now reaches U2.23 (CS)
- net \HAD: now reaches U2.3 (HAD)
- net \IRQ: now reaches U2.7 (IRQ)
- net LDS renamed \LDS
- net MLDS renamed \PLDS_M
- net MUDS renamed \PUDS_M
- net RW renamed R\W
- net UDS renamed \UDS
- net WIN renamed \WIN
Changed lines of the file:
@@
 $Descr A4 11693 8268
 encoding utf-8
-Sheet 1 4
+Sheet 1 6
 Title ""
 Date ""
@@
 $EndComp
 $Comp
-L 74xx:74LS00 U6
-U 1 1 5F49A598
-P 8950 2800
-F 0 "U6" H 8950 3125 50  0000 C CNN
-F 1 "74LS00" H 8950 3034 50  0000 C CNN
-F 2 "Package_SO:SOIC-14W_7.5x9mm_P1.27mm" H 8950 2800 50  0001 C CNN
-F 3 "http://www.ti.com/lit/gpn/sn74ls00" H 8950 2800 50  0001 C CNN
-	1    8950 2800
-	1    0    0    -1
-$EndComp
-$Comp
-L 74xx:74LS04 U5
-U 1 1 5F4A1C91
-P 8950 3350
-F 0 "U5" H 8950 3667 50  0000 C CNN
-F 1 "74LS04" H 8950 3576 50  0000 C CNN
-F 2 "Package_SO:SOIC-14_3.9x8.7mm_P1.27mm" H 8950 3350 50  0001 C CNN
-F 3 "http://www.ti.com/lit/gpn/sn74LS04" H 8950 3350 50  0001 C CNN
-	1    8950 3350
-	1    0    0    -1
-$EndComp
-$Comp
-L 74xx:74LS04 U5
-U 2 1 5F4A2E7E
-P 8950 3750
-F 0 "U5" H 8950 4067 50  0000 C CNN
-F 1 "74LS04" H 8950 3976 50  0000 C CNN
-F 2 "Package_SO:SOIC-14_3.9x8.7mm_P1.27mm" H 8950 3750 50  0001 C CNN
-F 3 "http://www.ti.com/lit/gpn/sn74LS04" H 8950 3750 50  0001 C CNN
-	2    8950 3750
-	1    0    0    -1
-$EndComp
-Text Label 9250 3350 0    50   ~ 0
-\MAS
-Text Label 9250 3750 0    50   ~ 0
-\AS
-Text Label 8650 2700 2    50   ~ 0
-\MAS
-Text Label 8650 2900 2    50   ~ 0
-\AS
-Text Label 9250 2800 0    50   ~ 0
-PAS
-$Comp
 L 74xx:74LS04 U5
 U 7 1 5F4AAA49
@@
 	1    0    0    -1
 $EndComp
-$Sheet
-S 4400 6400 1200 750
-U 5F4B6B1E
-F0 "PAD strobe" 50
-F1 "../file5F4B6B1D.sch" 50
-F2 "PUDS_R" U L 4400 6500 50
-F3 "PLDS_R" U L 4400 6600 50
-$EndSheet
-Text GLabel 5200 3500 0    50   Input ~ 0
-MUDS
-Text GLabel 5200 3600 0    50   Input ~ 0
-MLDS
-Text GLabel 4000 5350 2    50   BiDi ~ 0
-UDS
-Text GLabel 4000 5450 2    50   BiDi ~ 0
-LDS
-Text GLabel 4000 5550 2    50   BiDi ~ 0
-RW
+Text GLabel 4000 5350 2    50   Output ~ 0
+\UDS
+Text GLabel 4000 5450 2    50   Output ~ 0
+\LDS
+Text GLabel 4000 5550 2    50   Output ~ 0
+R\W
 Text GLabel 9850 4000 0    50   Input ~ 0
-RW
+R\W
 Text GLabel 9850 1900 0    50   Input ~ 0
-RW
+R\W
 Text GLabel 5200 5400 0    50   Input ~ 0
-RW
-Text GLabel 8650 3350 0    50   Input ~ 0
-MAS
+R\W
 Text GLabel 5200 4600 0    50   Output ~ 0
-MAS
+\MAS
 Text GLabel 5200 4300 0    50   Output ~ 0
-WIN
+\WIN
 $Sheet
 S 3150 6700 850  450
@@
 Connection ~ 8350 6200
 Connection ~ 8700 6200
-Text GLabel 2000 2350 0    50   BiDi ~ 0
+Text GLabel 2000 2350 0    50   Output ~ 0
 FC0
-Text GLabel 2000 2450 0    50   BiDi ~ 0
+Text GLabel 2000 2450 0    50   Output ~ 0
 FC1
-Text GLabel 2000 2550 0    50   BiDi ~ 0
+Text GLabel 2000 2550 0    50   Output ~ 0
 FC2
-Text GLabel 5200 1800 0    50   BiDi ~ 0
+Text GLabel 5200 1800 0    50   Input ~ 0
 FC0
-Text GLabel 5200 1900 0    50   BiDi ~ 0
+Text GLabel 5200 1900 0    50   Input ~ 0
 FC1
-Text GLabel 5200 2000 0    50   BiDi ~ 0
+Text GLabel 5200 2000 0    50   Input ~ 0
 FC2
-Text GLabel 8650 3750 0    50   Input ~ 0
-AS
-Text GLabel 5200 3400 0    50   BiDi ~ 0
-AS
+Text GLabel 5200 3400 0    50   Input ~ 0
+\AS
 Text GLabel 4000 5250 2    50   Output ~ 0
-AS
+\AS
 Text GLabel 2450 6550 0    50   UnSpc ~ 0
 ALL
@@
 Connection ~ 10300 6200
 Connection ~ 9950 6200
-Text Label 4400 6500 2    50   ~ 0
-PUDS_R
-Text Label 4400 6600 2    50   ~ 0
-PLDS_R
 Text Label 3150 6850 2    50   ~ 0
 ALL_R
@@
 Text Label 2450 6950 2    50   ~ 0
 MAS_R
-Text Label 2450 7050 2    50   ~ 0
-PUDS_R
-Text Label 2450 7150 2    50   ~ 0
-PLDS_R
 $Sheet
 S 6000 6600 700  500
@@
 F1 "mem.sch" 50
 $EndSheet
+Text GLabel 2000 1450 0    50   Input ~ 0
+\IPL0
+Text GLabel 2000 1550 0    50   Input ~ 0
+\IPL1
+Text GLabel 2000 1650 0    50   Input ~ 0
+\IPL2
+Text GLabel 2000 1850 0    50   Input ~ 0
+\BGACK
+Text GLabel 2000 1950 0    50   Output ~ 0
+\BG
+Text GLabel 2000 2050 0    50   Input ~ 0
+\BR
+Text GLabel 2000 2850 0    50   Output ~ 0
+\VMA
+Text GLabel 2000 2950 0    50   Output ~ 0
+E
+Text GLabel 2000 3050 0    50   Input ~ 0
+\VPA
+Text GLabel 2000 3950 0    50   Input ~ 0
+\BERR
+Text GLabel 2000 4550 0    50   BiDi ~ 0
+\HALT
+Text GLabel 2000 4650 0    50   BiDi ~ 0
+\RST
+Text GLabel 5200 1600 0    50   Input ~ 0
+\MMUSEL
+Text GLabel 5200 5100 0    50   Input ~ 0
+\RST
+Text GLabel 5200 3750 0    50   BiDi ~ 0
+\IRQ
+Text GLabel 5200 4800 0    50   BiDi ~ 0
+\BERR
+Text GLabel 5200 4500 0    50   Output ~ 0
+\HAD
+$Sheet
+S 4650 6650 1000 450
+U 601BFF66
+F0 "Physical data strobe" 50
+F1 "pds.sch" 50
+F2 "PUDS_R" O L 4650 6850 50
+F3 "PLDS_R" O L 4650 6950 50
+F4 "PUDS_M" O L 4650 6700 50
+F5 "PLDS_M" O L 4650 6750 50
+$EndSheet
+Text HLabel 5200 3600 0    50   Input ~ 0
+\PLDS_M
+Text HLabel 5200 3500 0    50   Input ~ 0
+\PUDS_M
+Text HLabel 2450 7050 0    50   Input ~ 0
+PUDS_R
+Text HLabel 2450 7150 0    50   Input ~ 0
+PLDS_R
+$Sheet
+S 4200 6000 500  350
+U 60229C16
+F0 "PAS Generator" 50
+F1 "pas_gen.sch" 50
+$EndSheet
+$Sheet
+S 3150 7350 600  300
+U 6037D76A
+F0 "External IO and MMUSEL" 50
+F1 "externio.sch" 50
+$EndSheet
 $EndSCHEMATC
