File: interrupthack.sch (KiCad schematic (older format))
At the start: 3 parts, among them U10 74LS05, U5 74LS04, U7 74LS08

Commit message: finish memory layout thing
Connections:
- net ALL renamed \ALL
- net AS renamed \AS
- net MAS renamed \MAS
Changed lines of the file:
@@
 $Descr A4 11693 8268
 encoding utf-8
-Sheet 3 4
+Sheet 2 6
 Title ""
 Date ""
@@
 FC2
 Text GLabel 4800 2150 0    50   Input ~ 0
-AS
+\AS
 $Comp
 L 74xx:74LS05 U10
@@
 	8300 2250 8300 1500
 Text GLabel 8700 1700 2    50   Output ~ 0
-MAS
+\MAS
 Text GLabel 8300 2250 2    50   Output ~ 0
-ALL
+\ALL
 Text HLabel 8300 1500 0    50   UnSpc ~ 0
 ALL_R
