File: mem.sch (KiCad schematic (older format))
At the start: 8 parts, among them U11 IS61C5128AS-25QLI, U12 IS61C5128AS-25QLI, U13 IS61C5128AS-25QLI, U14 IS61C5128AS-25QLI, U15 IS61C5128AS-25QLI, U16 IS61C5128AS-25QLI, U17 IS61C5128AS-25QLI, U18 IS61C5128AS-25QLI

Commit message: finish memory layout thing
Parts:
- removed U11, U12, U13, U14, U15, U16, U17, U18: IS61C5128AS-25QLI, Package_SO:SSOP-32_11.305x20.495mm_P1.27mm, symbol Memory_RAM:IS61C5128AS-25QLI
- added U? (x8): AS6C1616, Package_SO:TSOP-I-48_18.4x12mm_P0.5mm, symbol Memory_RAM:AS6C1616
- added U?: 74LS138, symbol 74xx:74LS138
- added U? (x2): 74LS10, symbol 74xx:74LS10
- added U? (x2): 74LS04, symbol 74xx:74LS04
- added U?: 74LS32, symbol 74xx:74LS32
Connections:
- net labels added: +5V, CS_MEMHI, DATA0, DATA1, DATA10, DATA11, DATA12, DATA13, DATA14, DATA15, DATA2, DATA3, DATA4, DATA5, DATA6, DATA7, DATA8, DATA9, FC2, GND, PA1, PA10, PA11, PA12, PA13, PA14, PA15, PA16, PA17, PA18, PA19, PA2, PA20, PA21, PA22, PA23, PA3, PA4, PA5, PA6, PA7, PA8, PA9, PAS, R\W, \CS_MEM0, \CS_MEM1, \CS_MEM2, \CS_MEM3, \CS_MEM4, \CS_MEM5, \CS_MEM6, \CS_MEM7, \CS_MEMHI, \MEMSEL_IO, \PLDS, \PUDS
